File: test_eyes.brd (EAGLE design)
At the start: 136 x 45 mm, 253 parts

Commit message: Removed half of decoupling caps for cost reduction
Parts:
- removed C1, C101, C103, C105, C107, C109, C11, C111, C113, C115, C117, C119, C121, C123, C125, C13, C14, C16, C18, C20, C23, C26, C28, C3, C31, C34, C36, C39, C4, C42, C44, C47, C49, C51, C52, C54, C57, C59, C6, C61, C63, C65, C67, C68, C70, C72, C74, C77, C79, C81, C83, C85, C87, C89, C9, C91, C93, C95, C97, C99: 0.1uF, SparkFun-Capacitors:0402
Connections:
- net GND: no longer C1.2, C101.2, C103.2, C105.2, C107.2, C109.2, C11.2, C111.2, C113.2, C115.2, C117.2, C119.2, C121.2, C123.2, C125.2, C13.2, C14.2, C16.2, C18.2, C20.2, C23.2, C26.2, C28.2, C3.2, C31.2, C34.2, C36.2, C39.2, C4.1, C42.2, C44.2, C47.2, C49.2, C51.2, C52.2, C54.2, C57.2, C59.2, C6.1, C61.2, C63.2, C65.2, C67.2, C68.2, C70.2, C72.2, C74.2, C77.2, C79.2, C81.2, C83.2, C85.2, C87.2, C89.2, C9.2, C91.2, C93.2, C95.2, C97.2, C99.2
- net VCC: no longer C1.1, C101.1, C103.1, C105.1, C107.1, C109.1, C11.1, C111.1, C113.1, C115.1, C117.1, C119.1, C121.1, C123.1, C125.1, C13.1, C14.1, C16.1, C18.1, C20.1, C23.1, C26.1, C28.1, C3.1, C31.1, C34.1, C36.1, C39.1, C4.2, C42.1, C44.1, C47.1, C49.1, C51.1, C52.1, C54.1, C57.1, C59.1, C6.2, C61.1, C63.1, C65.1, C67.1, C68.1, C70.1, C72.1, C74.1, C77.1, C79.1, C81.1, C83.1, C85.1, C87.1, C89.1, C9.1, C91.1, C93.1, C95.1, C97.1, C99.1
Routing:
- net VCC: track 1428.0 -> 1239.2 mm
